File: PCB/RocketPressurePID.kicad_pcb (KiCad board)
At the start: 2 copper layers, 47 parts, among them J1 TYPE-C 16PIN 2MD(073), J2 DW127R-22-14-23, J6 SM05B-SRSS-TB(LF)(SN), Q4 IRLML2502TRPBF, SW1 TS-1002S-08026C, SW2 TS-1002S-08026C, U2 HS HS13L03W2C01, U3 AMS1117-3.3, U4 M24C02-FMN, U5 STM32G030C8Tx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

Commit message: WIP
Parts:
- added D20: 5V_TVS, Diode_SMD:D_SOD-323, F.Cu at (148.4, 79.0)
- J2: value DW127R-22-14-23 -> 2x14 1.27mm SMD; footprint Connector_PinHeader_1.27mm:PinHeader_2x07_P1.27mm_Vertical -> Connector_PinHeader_1.27mm:PinHeader_2x07_P1.27mm_Vertical_SMD
- moved R8 60.8 mm to (138.5, 64.1)
- moved R7 55.5 mm to (121.2, 65.8), turned to -90 degrees
- moved D1 55.1 mm to (131.5, 71.8), turned to 180 degrees
- moved U3 50.5 mm to (129.8, 80.2), turned to 180 degrees
- moved C13 50.2 mm to (134.8, 68.8), turned to -90 degrees
- moved FB1 47.8 mm to (134.9, 72.5), turned to 90 degrees
- moved C14 45.3 mm to (132.3, 75.6), turned to 180 degrees
- moved D15 44.1 mm to (152.1, 104.4)
- moved U4 43.8 mm to (117.3, 80.3)
- moved C1 41.5 mm to (132.3, 73.8), turned to 180 degrees
- moved C15 39.8 mm to (103.7, 83.9), turned to 180 degrees
- moved C3 39.7 mm to (119.1, 76.7)
- moved C16 39.4 mm to (104.1, 86.7), turned to 180 degrees
- moved D16 39.2 mm to (152.1, 102.4)
- moved C2 38.8 mm to (135.3, 81.1), turned to -90 degrees
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Connections:
- D19 pad 1: /MCU_DBG_TX -> /MCU_DBG_RX
- J1 pad A1: (no net) -> GND
- J1 pad A4: (no net) -> Net-(D1-A)
- J1 pad B1: (no net) -> GND
- J1 pad B4: (no net) -> Net-(D1-A)
- SW1 pad 2: /~{SW_UP} -> GND
- SW2 pad 2: /~{SW_DOWN} -> GND
Routing:
- net +3.3V: track 0.00 -> 106.0 mm, vias 0 -> 3
- net /I2C_SCL: track 0.00 -> 42.7 mm, vias 0 -> 2
- net /I2C_SDA: track 0.00 -> 38.7 mm, vias 0 -> 2
- net Net-(D20-A1): track 0.00 -> 33.3 mm
- net +5V: track 0.00 -> 30.9 mm
- net /~{MCU_RESET}: track 0.00 -> 30.7 mm, vias 0 -> 2
- net /SSR_EN: track 0.00 -> 25.1 mm, vias 0 -> 2
- net /SWDIO: track 0.00 -> 18.0 mm, vias 0 -> 2
- net /SWCLK: track 0.00 -> 17.9 mm, vias 0 -> 2
- net Net-(D1-A): track 0.00 -> 15.2 mm
- net Net-(J6-Pin_5): track 0.00 -> 11.9 mm, vias 0 -> 2
- net Net-(U5-PF1): track 0.00 -> 9.22 mm
- net Net-(U5-PF0): track 0.00 -> 7.97 mm
- net /PRESSURE_IN_3V3: track 0.00 -> 6.89 mm
- net Net-(D1-K): track 0.00 -> 5.97 mm
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- added copper zone on B.Cu, net GND
- added copper zone on F.Cu, net GND
Other:
- board outline added: 58 x 47 mm

Commit message: WIP
Parts:
- J6: value SM05B-SRSS-TB(LF)(SN) -> S5B-PH-SM4-TB(LF)(SN); footprint Connector_JST:JST_SH_SM05B-SRSS-TB_1x05-1MP_P1.00mm_Horizontal -> Connector_JST:JST_PH_S5B-PH-SM4-TB_1x05-1MP_P2.00mm_Horizontal
- moved J6 2.30 mm to (155.9, 77.8)
Routing:
- net +5V: track 30.9 -> 15.5 mm
- net Net-(J6-Pin_5): track 11.9 -> 9.76 mm
- net Net-(D20-A1): track 33.3 -> 31.2 mm

Commit message: WIP
Parts:
- added R10: 0R, Resistor_SMD:R_0603_1608Metric, F.Cu at (130.8, 85.2)
- added R11: 0R, Resistor_SMD:R_0603_1608Metric, F.Cu at (155.3, 88.4)
- added R12: 0R, Resistor_SMD:R_0603_1608Metric, F.Cu at (153.7, 88.4)
- added R9: 0R, Resistor_SMD:R_0603_1608Metric, F.Cu at (131.8, 86.9)
- moved D15 21.4 mm to (137.8, 88.6), turned to 90 degrees
- moved D16 18.4 mm to (139.8, 88.6), turned to 90 degrees
- moved C15 10.5 mm to (113.8, 86.7)
- moved R3 10.5 mm to (113.8, 85.1)
- moved R4 10.2 mm to (112.5, 94.2)
- moved C16 10.2 mm to (112.5, 92.6)
- moved D20 9.38 mm to (149.3, 88.3), turned to 0 degrees
- moved R7 5.94 mm to (121.2, 71.7)
- moved J6 4.49 mm to (151.5, 78.3)
- moved D19 4.14 mm to (155.4, 92.8)
- moved J2 3.82 mm to (152.6, 99.9)
- moved D14 3.76 mm to (152.3, 91.3)
- moved D18 3.76 mm to (152.2, 93.4)
- moved C1 3.59 mm to (135.5, 75.5), turned to 0 degrees
- moved J1 3.44 mm to (128.0, 65.4)
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Connections:
- D18 pad 1: /MCU_DBG_TX -> Net-(D18-A1)
- D19 pad 1: /MCU_DBG_RX -> Net-(D19-A1)
- J2 pad 13: /MCU_DBG_RX -> Net-(D19-A1)
- J2 pad 14: /MCU_DBG_TX -> Net-(D18-A1)
Routing:
- net /~{SW_DOWN}: track 0.00 -> 48.5 mm, vias 0 -> 2
- net /~{SW_UP}: track 0.00 -> 47.1 mm, vias 0 -> 2
- net Net-(D19-A1): track 0.00 -> 37.4 mm, vias 0 -> 2
- net /MCU_DBG_RX: track 0.00 -> 35.3 mm, vias 0 -> 2
- net /MCU_DBG_TX: track 0.00 -> 32.5 mm, vias 0 -> 2
- net Net-(D18-A1): track 0.00 -> 31.0 mm, vias 0 -> 2
- net +5V: track 15.5 -> 40.5 mm
- net +3.3V: track 106.0 -> 130.9 mm, vias 3 -> 4
- net /SSR_EN: track 25.1 -> 36.1 mm, vias 2 -> 0
- net Net-(J1-CC2): track 0.00 -> 10.9 mm
- net /~{MCU_RESET}: track 30.7 -> 40.9 mm
- net Net-(J1-CC1): track 0.00 -> 9.11 mm
- net /SWDIO: track 18.0 -> 22.7 mm
- net /SWCLK: track 17.9 -> 21.6 mm
- net Net-(D1-A): track 15.2 -> 11.9 mm
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Other:
- board size 58 x 47 mm -> 54 x 42 mm
- board text added: "MYLA'S CIRCUIT BOARD"
- board text added: "PID Controller v1.0"

Commit message: v1.0 manufacturing
Parts:
- D1: value PMEG2010ER,115 -> ~
- moved D18 4.97 mm to (148.2, 90.4)
- moved D14 4.23 mm to (148.2, 92.5)
- moved C8 2.55 mm to (123.1, 86.9), turned to 0 degrees
- moved D19 2.40 mm to (153.2, 92.0), turned to 180 degrees
- moved C9 1.14 mm to (126.3, 89.0), turned to 180 degrees
- moved FB2 1.09 mm to (123.2, 85.3), turned to 180 degrees
- moved D20 1.08 mm to (148.2, 88.3)
Connections:
- C8 pad 1: Net-(U5-VREF+) -> GND
- C8 pad 2: Net-(C8-Pad2) -> Net-(U5-VREF+)
- FB2 pad 1: Net-(C8-Pad2) -> Net-(U5-VREF+)
Routing:
- net /~{MCU_RESET}: track 40.9 -> 33.9 mm
- net Net-(D18-A1): track 31.0 -> 36.7 mm
- net Net-(U5-VREF+): track 5.45 -> 10.3 mm
- net GND: track 3.88 -> 6.37 mm, vias 60 -> 62
- net +3.3V: track 130.9 -> 128.7 mm
- net Net-(C8-Pad2): track 1.55 -> 0.00 mm
- net Net-(D19-A1): track 37.4 -> 38.5 mm
- net Net-(D20-A1): track 33.0 -> 32.2 mm
- net /SSR_EN: track 36.1 -> 35.6 mm
Other:
- outline, holes or cut-outs redrawn
- board text added: "1"
- board text added: "1 - Sense 5V"
- board text added: "2 - Sense SIG"
- board text added: "3 - Sense GND"
- board text added: "4 - SSR (+)"
- board text added: "5"
- board text added: "5 - SSR (-)"
