File: PCB/RocketPressurePID.kicad_sch (KiCad schematic)
At the start: 47 parts, among them J1 TYPE-C 16PIN 2MD(073), J2 DW127R-22-14-23, J6 SM05B-SRSS-TB(LF)(SN), Q4 IRLML2502TRPBF, SW1 TS-1002S-08026C, SW2 TS-1002S-08026C, U2 HS HS13L03W2C01, U3 AMS1117-3.3, U4 M24C02-FMN, U5 STM32G030C8Tx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

Commit message: WIP
Parts:
- removed U2: HS HS13L03W2C01, project:HS13L03W2C01, symbol Display_Graphic:ER_OLEDM0.91_1x-I2C
- added D20: 5V_TVS, Diode_SMD:D_SOD-323, symbol Device:D_TVS_ALT
- J1: symbol Connector:USB_C_Receptacle_PowerOnly_6P -> Connector:USB_C_Receptacle_PowerOnly_24P
- J2: value DW127R-22-14-23 -> 2x14 1.27mm SMD; footprint Connector_PinHeader_1.27mm:PinHeader_2x07_P1.27mm_Vertical -> Connector_PinHeader_1.27mm:PinHeader_2x07_P1.27mm_Vertical_SMD; LCSC C2935955 -> C41376039
- J5: now not fitted
- SW1, SW2: symbol Switch:SW_MEC_5E -> project:SW_MEC
Connections:
- net GND: now also J1.A1 (GND), J1.B1 (GND), SW1.2, SW2.2, D20.2 (A2); no longer SW1.3 (K), SW1.4 (A), SW2.3 (K), SW2.4 (A)
- net MCU_DBG_RX: now also D19.1 (A1)
- net MCU_DBG_TX: no longer D19.1 (A1)
- net ~{SW_DOWN}: no longer SW2.2
- net ~{SW_UP}: no longer SW1.2
- net at J6.2 (Pin_2), R6.1: now also D20.1 (A1)
- net at D1.2 (A), J1.A9 (VBUS), J1.B9 (VBUS): now also J1.A4 (VBUS), J1.B4 (VBUS)
Other:
- note added: "2.54mm Headers to HS HS13L03W2C01 OLED"
- note added: "DOWN Button"
- note added: "MCU"
- note added: "Pin 1: Pressure Sensor 5V IN Pin 2: Pressure Sensor SIG OUT Pin 3: Pressure Sensor GND Pin 4: SSR EN HIGH Pin 5: SSR EN LOW"
- note added: "UP Button"
- note removed: "2.54mm Headers to OLED"
- note removed: "DOWN"
- note removed: "I2C OLED with SH1106"
- note removed: "Pressure sensor 5V to 3.3V divider"
- note removed: "TODO: verify these threads will fit"
- note removed: "To SSR https://a.co/d/04Bq4Fb9"
- note removed: "UP"
- moved on the sheet: C1, C10, C11, C12, C13, C15, C16, C17, C18, C19, C3, C8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

Commit message: WIP
Parts:
- J6: value SM05B-SRSS-TB(LF)(SN) -> S5B-PH-SM4-TB(LF)(SN); footprint Connector_JST:JST_SH_SM05B-SRSS-TB_1x05-1MP_P1.00mm_Horizontal -> Connector_JST:JST_PH_S5B-PH-SM4-TB_1x05-1MP_P2.00mm_Horizontal; LCSC C136657 -> C265104
Other:
- note removed: "Digikey pigtail: 455-3711-ND"
Changed lines of the file:
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@@
 		)
 	)
-	(text "Digikey pigtail:\n455-3711-ND"
-		(exclude_from_sim no)
-		(at 259.588 76.073 0)
-		(effects
-			(font
-				(size 1.27 1.27)
-			)
-		)
-	)
 	(text "5V to 3.3V LDO"
 		(exclude_from_sim no)
@@
 			)
 		)
-		(property "Value" "SM05B-SRSS-TB(LF)(SN)"
+		(property "Value" "S5B-PH-SM4-TB(LF)(SN)"
 			(at 252.73 70.4849 0)
 			(show_name no)
@@
 			)
 		)
-		(property "Footprint" "Connector_JST:JST_SH_SM05B-SRSS-TB_1x05-1MP_P1.00mm_Horizontal"
+		(property "Footprint" "Connector_JST:JST_PH_S5B-PH-SM4-TB_1x05-1MP_P2.00mm_Horizontal"
 			(at 249.555 69.215 0)
 			(hide yes)
@@
 			)
 		)
-		(property "LCSC" "C136657"
+		(property "LCSC" "C265104"
 			(at 249.555 69.215 0)
 			(hide yes)

Commit message: WIP
Parts:
- added R10, R11, R12, R9: 0R, Resistor_SMD:R_0603_1608Metric, symbol Device:R_Small
Connections:
- net MCU_DBG_RX: now also R10.1, R12.1; no longer D19.1 (A1), J2.13
- net MCU_DBG_TX: now also R11.1, R9.1; no longer D18.1 (A1), J2.14
- new net: D19.1 (A1), J2.13, R10.2, R11.2
- new net: D18.1 (A1), J2.14, R12.2, R9.2
Other:
- note added: "In case TX/RX are swapped"
- moved on the sheet: D14, D15, D16, D18, D19, J2

Commit message: v1.0 manufacturing
Parts:
- C1: LCSC C2762594 -> C59461
- C17, C18: LCSC C113797 -> C1658
- D1: value PMEG2010ER,115 -> (none); LCSC C82288 -> C8598
- FB1, FB2: LCSC C88984 -> C1002
- J2: Manufacturer DEALON -> (none); Part Number DW127R-22-14-23 -> (none)
- R1, R3, R4, R5: LCSC C116677 -> C25804
- R10, R11, R12, R9: LCSC C95177 -> C21189
- R6, R7, R8: LCSC C105580 -> C23186
- STD1, STD2, STD3: Alt MPN (none) -> 9774040151R
- U5: LCSC (none) -> C529329
Connections:
- net GND: now also C8.1
- net at U5.5 (VREF+): now also C8.2, FB2.1; no longer C8.1
- no-connect marks 6 -> 35
Other:
- moved on the sheet: C8, FB2

Commit message: Updated alt part number
Parts:
- STD4: Alt MPN (none) -> 9774040151R
Changed lines of the file:
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@@
 			)
 		)
-		(property "Alt MPN" ""
+		(property "Alt MPN" "9774040151R"
 			(at 202.565 24.13 0)
 			(hide yes)
